Commit message: 机械臂铲子配置

File: src/ur10_description/urdf/ur10_sim.urdf.xacro (robot description, xacro)
@@ -210,4 +210,61 @@
     <origin xyz="0 0 0" rpy="0 0 0"/>
   </joint>
+  <link name="gantry_depth_camera_link">
+    <visual name="gantry_depth_camera_visual">
+      <origin xyz="0 0 0" rpy="0 0 0"/>
+      <geometry>
+        <box size="0.10 0.06 0.05"/>
+      </geometry>
+      <material name="depth_camera_black">
+        <color rgba="0.08 0.08 0.10 1.0"/>
+      </material>
+    </visual>
+    <collision name="gantry_depth_camera_collision">
+      <origin xyz="0 0 0" rpy="0 0 0"/>
+      <geometry>
+        <box size="0.10 0.06 0.05"/>
+      </geometry>
+    </collision>
+    <xacro:box_inertial x="0.10" y="0.06" z="0.05" mass="0.4"/>
+  </link>
+  <joint name="gantry_depth_camera_joint" type="fixed">
+    <parent link="gantry_structure_link"/>
+    <child link="gantry_depth_camera_link"/>
+    <origin xyz="0 0 $(arg gantry_base_height)" rpy="0 -1.57079632679 0"/>
+  </joint>
+  <gazebo reference="gantry_depth_camera_link">
+    <sensor type="depth" name="gantry_depth_camera_sensor">
+      <update_rate>15.0</update_rate>
+      <visualize>false</visualize>
+      <pose>0 0 -0.10 0 0 0</pose>
+      <camera>
+        <horizontal_fov>1.25</horizontal_fov>
+        <image>
+          <width>640</width>
+          <height>480</height>
+          <format>B8G8R8</format>
+        </image>
+        <depth_camera/>
+        <clip>
+          <near>0.10</near>
+          <far>4.00</far>
+        </clip>
+      </camera>
+      <plugin name="gantry_depth_camera_plugin" filename="libgazebo_ros_camera.so">
+        <ros>
+          <namespace>/gantry_depth_camera</namespace>
+          <remapping>gantry_depth_camera/image_raw:=image_raw</remapping>
+          <remapping>gantry_depth_camera/camera_info:=camera_info</remapping>
+          <remapping>gantry_depth_camera/depth/image_raw:=depth/image_raw</remapping>
+          <remapping>gantry_depth_camera/depth/camera_info:=depth/camera_info</remapping>
+          <remapping>gantry_depth_camera/points:=points</remapping>
+        </ros>
+        <camera_name>gantry_depth_camera</camera_name>
+        <frame_name>gantry_depth_camera_link</frame_name>
+        <min_depth>0.10</min_depth>
+        <max_depth>4.00</max_depth>
+      </plugin>
+    </sensor>
+  </gazebo>
   <ros2_control name="gantry" type="system">
     <hardware>
