Commit message: Add gantry simulation launch file and URDF definitions for my_robot
- Created a new launch file `sim_planning_gantry.launch.py` to set up the simulation environment for the gantry robot, including integration with Gazebo and MoveIt.
- Added a new URDF file `my_robot_gantry.urdf.xacro` defining the structure and joints of the gantry robot, including visual and collision properties.
- Introduced a macro file `my_robot_macro.urdf.xacro` to encapsulate the robot model definition, including joint configurations and transmission settings for different hardware interfaces.

File: src/my_robot_xacro/my_robot/my_robot.urdf.xacro (robot description, xacro)
@@ -1,582 +1,11 @@
 <?xml version="1.0"?>
 <robot name="my_robot" xmlns:xacro="http://www.ros.org/wiki/xacro">
-  <link name="ur10">
-    <visual>
-      <origin xyz="0 0 0" rpy="0 0 0" />
-      <geometry>
-        <mesh filename="package://my_robot/meshes/base.dae" />
-      </geometry>
-    </visual>
-    <collision>
-      <origin xyz="0 0 0.019" rpy="0 0 0" />
-      <geometry>
-        <cylinder radius="0.075" length="0.038" />
-      </geometry>
-    </collision>
-    <inertial>
-      <origin xyz="0 0 0" rpy="0 0 0" />
-      <mass value="4" />
-      <inertia ixx="0.0061063" ixy="0" ixz="0" iyy="0.0061063" iyz="0" izz="0.01125" />
-    </inertial>
-  </link>
-  <link name="ur10_shoulder">
-    <visual>
-      <origin xyz="0 0 0" rpy="0 0 0" />
-      <geometry>
-        <mesh filename="package://my_robot/meshes/shoulder.dae" />
-      </geometry>
-    </visual>
-    <collision>
-      <origin xyz="0 0 0" rpy="0 0 0" />
-      <geometry>
-        <cylinder radius="0.075" length="0.177" />
-      </geometry>
-    </collision>
-    <inertial>
-      <origin xyz="0 0 0" rpy="0 0 0" />
-      <mass value="7.778" />
-      <inertia ixx="0.0314743" ixy="0" ixz="0" iyy="0.0314743" iyz="0" izz="0.0218756" />
-    </inertial>
-  </link>
-  <link name="ur10_upper_arm">
-    <visual>
-      <origin xyz="0 0 0" rpy="0 0 0" />
-      <geometry>
-        <mesh filename="package://my_robot/meshes/upperarm.dae" />
-      </geometry>
-    </visual>
-    <collision>
-      <origin xyz="0 -0.045 0" rpy="1.5707 0 0" />
-      <geometry>
-        <cylinder radius="0.075" length="0.177" />
-      </geometry>
-    </collision>
-    <collision>
-      <origin xyz="0 -0.0436 0.32" rpy="0 0 1.5707" />
-      <geometry>
-        <cylinder radius="0.058" length="0.461" />
-      </geometry>
-    </collision>
-    <collision>
-      <origin xyz="0 -0.04 0.613" rpy="1.5707 0 0" />
-      <geometry>
-        <cylinder radius="0.058" length="0.129" />
-      </geometry>
-    </collision>
-    <inertial>
-      <origin xyz="0 0 0.306" rpy="0 0 0" />
-      <mass value="12.93" />
-      <inertia ixx="0.421754" ixy="0" ixz="0" iyy="0.421754" iyz="0" izz="0.0363656" />
-    </inertial>
-  </link>
-  <link name="ur10_forearm">
-    <visual>
-      <origin xyz="0 0 0" rpy="0 0 0" />
-      <geometry>
-        <mesh filename="package://my_robot/meshes/forearm.dae" />
-      </geometry>
-    </visual>
-    <collision>
-      <origin xyz="0 0 0.001" rpy="1.5707 0 0" />
-      <geometry>
-        <cylinder radius="0.058" length="0.136" />
-      </geometry>
-    </collision>
-    <collision>
-      <origin xyz="0 0 0.305" rpy="0 0 1.5707" />
-      <geometry>
-        <cylinder radius="0.045" length="0.447" />
-      </geometry>
-    </collision>
-    <collision>
-      <origin xyz="0 0.001 0.5735" rpy="1.5707 0 0" />
-      <geometry>
-        <cylinder radius="0.045" length="0.119" />
-      </geometry>
-    </collision>
-    <inertial>
-      <origin xyz="0 0 0.28615" rpy="0 0 0" />
-      <mass value="3.87" />
-      <inertia ixx="0.11107" ixy="0" ixz="0" iyy="0.11107" iyz="0" izz="0.0108844" />
-    </inertial>
-  </link>
-  <link name="ur10_wrist_1">
-    <visual>
-      <origin xyz="0 0 0" rpy="0 0 0" />
-      <geometry>
-        <mesh filename="package://my_robot/meshes/wrist1.dae" />
-      </geometry>
-    </visual>
-    <collision>
-      <origin xyz="0 0.115 0.0025" rpy="0 0 0" />
-      <geometry>
-        <cylinder radius="0.0455" length="0.119" />
-      </geometry>
-    </collision>
-    <inertial>
-      <origin xyz="0 0 0" rpy="0 0 0" />
-      <mass value="1.96" />
-      <inertia ixx="0.0051082" ixy="0" ixz="0" iyy="0.0051082" iyz="0" izz="0.0055125" />
-    </inertial>
-  </link>
-  <link name="ur10_wrist_2">
-    <visual>
-      <origin xyz="0 0 0" rpy="0 0 0" />
-      <geometry>
-        <mesh filename="package://my_robot/meshes/wrist2.dae" />
-      </geometry>
-    </visual>
-    <collision>
-      <origin xyz="0 0.002 0.11659" rpy="1.5707 0 0" />
-      <geometry>
-        <cylinder radius="0.0455" length="0.119" />
-      </geometry>
-    </collision>
-    <inertial>
-      <origin xyz="0 0 0" rpy="0 0 0" />
-      <mass value="1.96" />
-      <inertia ixx="0.0051082" ixy="0" ixz="0" iyy="0.0051082" iyz="0" izz="0.0055125" />
-    </inertial>
-  </link>
-  <link name="ur10_wrist_3">
-    <visual>
-      <origin xyz="0 0 0" rpy="0 0 0" />
-      <geometry>
-        <mesh filename="package://my_robot/meshes/wrist3.dae" />
-      </geometry>
-    </visual>
-    <collision>
-      <origin xyz="0 0.0765 0" rpy="1.5707 0 0" />
-      <geometry>
-        <cylinder radius="0.045" length="0.031" />
-      </geometry>
-    </collision>
-    <inertial>
-      <origin xyz="0 0 0" rpy="0 0 0" />
-      <mass value="0.202" />
-      <inertia ixx="0.0005265" ixy="0" ixz="0" iyy="0.0005265" iyz="0" izz="0.0005681" />
-    </inertial>
-  </link>
-  <link name="铲子">
-    <visual>
-      <origin xyz="0 0 0" rpy="0 0 0" />
-      <geometry>
-        <mesh filename="package://my_robot/meshes/base_link.STL" />
-      </geometry>
-      <material name="铲子_mat">
-        <color rgba="0.64706275 0.61961176 0.58823922 1.00000000"/>
-      </material>
-    </visual>
-    <collision>
-      <origin xyz="0 0 0" rpy="0 0 0" />
-      <geometry>
-        <mesh filename="package://my_robot/meshes/base_link.STL" />
-      </geometry>
-    </collision>
-    <inertial>
-      <origin xyz="0.0002787 0.0006902 -0.1177" rpy="0 0 0" />
-      <mass value="1.512" />
-      <inertia ixx="0.0070805" ixy="-0.0000053" ixz="0.0002891" iyy="0.0068883" iyz="0.0000875" izz="0.0004825" />
-    </inertial>
-  </link>
-  <joint name="ur10_shoulder_pan" type="revolute">
-    <parent link="ur10" />
-    <child link="ur10_shoulder" />
-    <origin xyz="0 0 0.1273" rpy="0 0 0" />
-    <axis xyz="0 0 1" />
-    <limit lower="-6.28319" upper="6.28319" effort="330" velocity="2.16" />
-  </joint>
-  <joint name="ur10_shoulder_lift" type="revolute">
-    <parent link="ur10_shoulder" />
-    <child link="ur10_upper_arm" />
-    <origin xyz="0 0.220941 0" rpy="0 1.57079 0" />
-    <axis xyz="0 1 0" />
-    <limit lower="-6.28319" upper="6.28319" effort="330" velocity="2.16" />
-  </joint>
-  <joint name="ur10_elbow" type="revolute">
-    <parent link="ur10_upper_arm" />
-    <child link="ur10_forearm" />
-    <origin xyz="-0.0000039 -0.1719 0.612" rpy="0 0 0" />
-    <axis xyz="0 1 0" />
-    <limit lower="-6.28319" upper="6.28319" effort="150" velocity="3.15" />
-  </joint>
-  <joint name="ur10_wrist_1" type="revolute">
-    <parent link="ur10_forearm" />
-    <child link="ur10_wrist_1" />
-    <origin xyz="-0.0000036 0 0.5723" rpy="0 1.5707895 0.0000027" />
-    <axis xyz="0 1 0" />
-    <limit lower="-6.28319" upper="6.28319" effort="54" velocity="3.2" />
-  </joint>
-  <joint name="ur10_wrist_2" type="revolute">
-    <parent link="ur10_wrist_1" />
-    <child link="ur10_wrist_2" />
-    <origin xyz="0.0000003 0.1149 0.0000003" rpy="0 0 0" />
-    <axis xyz="0 0 -1" />
-    <limit lower="-6.28319" upper="6.28319" effort="54" velocity="3.2" />
-  </joint>
-  <joint name="ur10_wrist_3" type="revolute">
-    <parent link="ur10_wrist_2" />
-    <child link="ur10_wrist_3" />
-    <origin xyz="0 -0.0000003 0.1157" rpy="0 0 0" />
-    <axis xyz="0 1 0" />
-    <limit lower="-6.28319" upper="6.28319" effort="54" velocity="3.2" />
-  </joint>
-  <joint name="ur10-robot" type="fixed">
-    <parent link="ur10_wrist_3" />
-    <child link="铲子" />
-    <origin xyz="0 0.105 0" rpy="1.5707963 0 -1.5707963" />
-  </joint>
   <xacro:arg name="ros_profile" default="ros2" />
   <xacro:arg name="ros_hardware_interface" default="position" />
-  <xacro:if value="${xacro.arg('ros_profile') == 'ros1' and xacro.arg('ros_hardware_interface') == 'effort'}">
-      <transmission name="ur10_shoulder_pan_trans">
-        <type>transmission_interface/SimpleTransmission</type>
-        <joint name="ur10_shoulder_pan">
-          <hardwareInterface>hardware_interface/EffortJointInterface</hardwareInterface>
-        </joint>
-        <actuator name="ur10_shoulder_pan_motor">
-          <hardwareInterface>hardware_interface/EffortJointInterface</hardwareInterface>
-          <mechanicalReduction>1</mechanicalReduction>
-        </actuator>
-      </transmission>
-      <transmission name="ur10_shoulder_lift_trans">
-        <type>transmission_interface/SimpleTransmission</type>
-        <joint name="ur10_shoulder_lift">
-          <hardwareInterface>hardware_interface/EffortJointInterface</hardwareInterface>
-        </joint>
-        <actuator name="ur10_shoulder_lift_motor">
-          <hardwareInterface>hardware_interface/EffortJointInterface</hardwareInterface>
-          <mechanicalReduction>1</mechanicalReduction>
-        </actuator>
-      </transmission>
-      <transmission name="ur10_elbow_trans">
-        <type>transmission_interface/SimpleTransmission</type>
-        <joint name="ur10_elbow">
-          <hardwareInterface>hardware_interface/EffortJointInterface</hardwareInterface>
-        </joint>
-        <actuator name="ur10_elbow_motor">
-          <hardwareInterface>hardware_interface/EffortJointInterface</hardwareInterface>
-          <mechanicalReduction>1</mechanicalReduction>
-        </actuator>
-      </transmission>
-      <transmission name="ur10_wrist_1_trans">
-        <type>transmission_interface/SimpleTransmission</type>
-        <joint name="ur10_wrist_1">
-          <hardwareInterface>hardware_interface/EffortJointInterface</hardwareInterface>
-        </joint>
-        <actuator name="ur10_wrist_1_motor">
-          <hardwareInterface>hardware_interface/EffortJointInterface</hardwareInterface>
-          <mechanicalReduction>1</mechanicalReduction>
-        </actuator>
-      </transmission>
-      <transmission name="ur10_wrist_2_trans">
-        <type>transmission_interface/SimpleTransmission</type>
-        <joint name="ur10_wrist_2">
-          <hardwareInterface>hardware_interface/EffortJointInterface</hardwareInterface>
-        </joint>
-        <actuator name="ur10_wrist_2_motor">
-          <hardwareInterface>hardware_interface/EffortJointInterface</hardwareInterface>
-          <mechanicalReduction>1</mechanicalReduction>
-        </actuator>
-      </transmission>
-      <transmission name="ur10_wrist_3_trans">
-        <type>transmission_interface/SimpleTransmission</type>
-        <joint name="ur10_wrist_3">
-          <hardwareInterface>hardware_interface/EffortJointInterface</hardwareInterface>
-        </joint>
-        <actuator name="ur10_wrist_3_motor">
-          <hardwareInterface>hardware_interface/EffortJointInterface</hardwareInterface>
-          <mechanicalReduction>1</mechanicalReduction>
-        </actuator>
-      </transmission>
-      <gazebo>
-        <plugin name="gazebo_ros_control" filename="libgazebo_ros_control.so">
-          <robotNamespace>/my_robot_gazebo</robotNamespace>
-          <robotSimType>gazebo_ros_control/DefaultRobotHWSim</robotSimType>
-        </plugin>
-      </gazebo>
-  </xacro:if>
-  <xacro:if value="${xacro.arg('ros_profile') == 'ros1' and xacro.arg('ros_hardware_interface') == 'position'}">
-      <transmission name="ur10_shoulder_pan_trans">
-        <type>transmission_interface/SimpleTransmission</type>
-        <joint name="ur10_shoulder_pan">
-          <hardwareInterface>hardware_interface/PositionJointInterface</hardwareInterface>
-        </joint>
-        <actuator name="ur10_shoulder_pan_motor">
-          <hardwareInterface>hardware_interface/PositionJointInterface</hardwareInterface>
-          <mechanicalReduction>1</mechanicalReduction>
-        </actuator>
-      </transmission>
-      <transmission name="ur10_shoulder_lift_trans">
-        <type>transmission_interface/SimpleTransmission</type>
-        <joint name="ur10_shoulder_lift">
-          <hardwareInterface>hardware_interface/PositionJointInterface</hardwareInterface>
-        </joint>
-        <actuator name="ur10_shoulder_lift_motor">
-          <hardwareInterface>hardware_interface/PositionJointInterface</hardwareInterface>
-          <mechanicalReduction>1</mechanicalReduction>
-        </actuator>
-      </transmission>
-      <transmission name="ur10_elbow_trans">
-        <type>transmission_interface/SimpleTransmission</type>
-        <joint name="ur10_elbow">
-          <hardwareInterface>hardware_interface/PositionJointInterface</hardwareInterface>
-        </joint>
-        <actuator name="ur10_elbow_motor">
-          <hardwareInterface>hardware_interface/PositionJointInterface</hardwareInterface>
-          <mechanicalReduction>1</mechanicalReduction>
-        </actuator>
-      </transmission>
-      <transmission name="ur10_wrist_1_trans">
-        <type>transmission_interface/SimpleTransmission</type>
-        <joint name="ur10_wrist_1">
-          <hardwareInterface>hardware_interface/PositionJointInterface</hardwareInterface>
-        </joint>
-        <actuator name="ur10_wrist_1_motor">
-          <hardwareInterface>hardware_interface/PositionJointInterface</hardwareInterface>
-          <mechanicalReduction>1</mechanicalReduction>
-        </actuator>
-      </transmission>
-      <transmission name="ur10_wrist_2_trans">
-        <type>transmission_interface/SimpleTransmission</type>
-        <joint name="ur10_wrist_2">
-          <hardwareInterface>hardware_interface/PositionJointInterface</hardwareInterface>
-        </joint>
-        <actuator name="ur10_wrist_2_motor">
-          <hardwareInterface>hardware_interface/PositionJointInterface</hardwareInterface>
-          <mechanicalReduction>1</mechanicalReduction>
-        </actuator>
-      </transmission>
-      <transmission name="ur10_wrist_3_trans">
-        <type>transmission_interface/SimpleTransmission</type>
-        <joint name="ur10_wrist_3">
-          <hardwareInterface>hardware_interface/PositionJointInterface</hardwareInterface>
-        </joint>
-        <actuator name="ur10_wrist_3_motor">
-          <hardwareInterface>hardware_interface/PositionJointInterface</hardwareInterface>
-          <mechanicalReduction>1</mechanicalReduction>
-        </actuator>
-      </transmission>
-      <gazebo>
-        <plugin name="gazebo_ros_control" filename="libgazebo_ros_control.so">
-          <robotNamespace>/my_robot_gazebo</robotNamespace>
-          <robotSimType>gazebo_ros_control/DefaultRobotHWSim</robotSimType>
-        </plugin>
-      </gazebo>
-  </xacro:if>
-  <xacro:if value="${xacro.arg('ros_profile') == 'ros1' and xacro.arg('ros_hardware_interface') == 'velocity'}">
-      <transmission name="ur10_shoulder_pan_trans">
-        <type>transmission_interface/SimpleTransmission</type>
-        <joint name="ur10_shoulder_pan">
-          <hardwareInterface>hardware_interface/VelocityJointInterface</hardwareInterface>
-        </joint>
-        <actuator name="ur10_shoulder_pan_motor">
-          <hardwareInterface>hardware_interface/VelocityJointInterface</hardwareInterface>
-          <mechanicalReduction>1</mechanicalReduction>
-        </actuator>
-      </transmission>
-      <transmission name="ur10_shoulder_lift_trans">
-        <type>transmission_interface/SimpleTransmission</type>
-        <joint name="ur10_shoulder_lift">
-          <hardwareInterface>hardware_interface/VelocityJointInterface</hardwareInterface>
-        </joint>
-        <actuator name="ur10_shoulder_lift_motor">
-          <hardwareInterface>hardware_interface/VelocityJointInterface</hardwareInterface>
-          <mechanicalReduction>1</mechanicalReduction>
-        </actuator>
-      </transmission>
-      <transmission name="ur10_elbow_trans">
-        <type>transmission_interface/SimpleTransmission</type>
-        <joint name="ur10_elbow">
-          <hardwareInterface>hardware_interface/VelocityJointInterface</hardwareInterface>
-        </joint>
-        <actuator name="ur10_elbow_motor">
-          <hardwareInterface>hardware_interface/VelocityJointInterface</hardwareInterface>
-          <mechanicalReduction>1</mechanicalReduction>
-        </actuator>
-      </transmission>
-      <transmission name="ur10_wrist_1_trans">
-        <type>transmission_interface/SimpleTransmission</type>
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