Commit message: docs: 重写项目 README，并补充功能包分析与 Gazebo 排障文档

File: src/my_robot_moveit_config/srdf/my_robot.srdf.xacro (robot description, xacro)
@@ -43,6 +43,6 @@
   <disable_collisions link1="ur10_wrist_1" link2="ur10_wrist_2" reason="Adjacent" />
   <disable_collisions link1="ur10_wrist_2" link2="ur10_wrist_3" reason="Adjacent" />
-  <disable_collisions link1="ur10_wrist_3" link2="铲子" reason="Adjacent" />
+  <disable_collisions link1="ur10_wrist_3" link2="shovel_link" reason="Adjacent" />
   <disable_collisions link1="ur10_wrist_3" link2="shovel_tip" reason="Adjacent" />
-  <disable_collisions link1="铲子" link2="shovel_tip" reason="Never" />
+  <disable_collisions link1="shovel_link" link2="shovel_tip" reason="Never" />
 </robot>

File: src/my_robot_xacro/my_robot/my_robot.urdf.xacro (robot description, xacro)
@@ -4,5 +4,5 @@
   <xacro:arg name="ros_hardware_interface" default="position" />
   <xacro:arg name="inject_gazebo_ros_control_plugin" default="true" />
-  <xacro:arg name="use_gazebo_compatible_visuals" default="false" />
+  <xacro:arg name="use_gazebo_visual_meshes" default="false" />
   <xacro:include filename="$(find my_robot)/urdf/my_robot_macro.urdf.xacro" />
   <xacro:my_robot_model
@@ -10,4 +10,4 @@
     ros_hardware_interface="$(arg ros_hardware_interface)"
     inject_gazebo_ros_control_plugin="$(arg inject_gazebo_ros_control_plugin)"
-    use_gazebo_compatible_visuals="$(arg use_gazebo_compatible_visuals)" />
+    use_gazebo_visual_meshes="$(arg use_gazebo_visual_meshes)" />
 </robot>

File: src/my_robot_xacro/my_robot/urdf/my_robot_gantry.urdf.xacro (robot description, xacro)
@@ -15,5 +15,5 @@
   <xacro:arg name="gantry_z_max" default="0.0" />
   <xacro:arg name="gantry_base_height" default="2.2" />
-  <xacro:arg name="use_gazebo_compatible_visuals" default="true" />
+  <xacro:arg name="use_gazebo_visual_meshes" default="true" />
   <xacro:include filename="$(find my_robot)/urdf/my_robot_macro.urdf.xacro" />
   <xacro:macro name="box_inertial" params="x y z mass">
@@ -201,9 +201,40 @@
     ros_hardware_interface="$(arg ros_hardware_interface)"
     inject_gazebo_ros_control_plugin="false"
-    use_gazebo_compatible_visuals="$(arg use_gazebo_compatible_visuals)" />
-  <ros2_control name="gantry" type="system">
+    include_ros2_control="false"
+    use_gazebo_visual_meshes="$(arg use_gazebo_visual_meshes)" />
+  <ros2_control name="my_robot_gantry" type="system">
     <hardware>
       <plugin>gazebo_ros2_control/GazeboSystem</plugin>
     </hardware>
+    <joint name="ur10_shoulder_pan">
+      <command_interface name="position" />
+      <state_interface name="position" />
+      <state_interface name="velocity" />
+    </joint>
+    <joint name="ur10_shoulder_lift">
+      <command_interface name="position" />
+      <state_interface name="position" />
+      <state_interface name="velocity" />
+    </joint>
+    <joint name="ur10_elbow">
+      <command_interface name="position" />
+      <state_interface name="position" />
+      <state_interface name="velocity" />
+    </joint>
+    <joint name="ur10_wrist_1_joint">
+      <command_interface name="position" />
+      <state_interface name="position" />
+      <state_interface name="velocity" />
+    </joint>
+    <joint name="ur10_wrist_2_joint">
+      <command_interface name="position" />
+      <state_interface name="position" />
+      <state_interface name="velocity" />
+    </joint>
+    <joint name="ur10_wrist_3_joint">
+      <command_interface name="position" />
+      <state_interface name="position" />
+      <state_interface name="velocity" />
+    </joint>
     <joint name="gantry_x_joint">
       <command_interface name="position" />

File: src/my_robot_xacro/my_robot/urdf/my_robot_macro.urdf.xacro (robot description, xacro)
@@ -3,25 +3,19 @@
   <xacro:macro
     name="my_robot_model"
-    params="ros_profile:='ros2' ros_hardware_interface:='position' inject_gazebo_ros_control_plugin:='true' use_gazebo_compatible_visuals:='false'">
-  <xacro:macro name="ur_gray_material" params="name rgba">
-    <material name="${name}">
-      <color rgba="${rgba}" />
-    </material>
-  </xacro:macro>
-  <xacro:macro name="ur_visual_or_gazebo_cylinder" params="mesh_filename radius length origin_xyz origin_rpy material_name material_rgba">
-    <xacro:if value="${use_gazebo_compatible_visuals}">
-      <visual>
-        <origin xyz="${origin_xyz}" rpy="${origin_rpy}" />
-        <geometry>
-          <cylinder radius="${radius}" length="${length}" />
-        </geometry>
-        <xacro:ur_gray_material name="${material_name}" rgba="${material_rgba}" />
-      </visual>
-    </xacro:if>
-    <xacro:unless value="${use_gazebo_compatible_visuals}">
+    params="ros_profile:='ros2' ros_hardware_interface:='position' inject_gazebo_ros_control_plugin:='true' include_ros2_control:='true' use_gazebo_visual_meshes:='false'">
+  <xacro:macro name="ur_visual_mesh" params="dae_mesh stl_mesh">
+    <xacro:if value="${use_gazebo_visual_meshes}">
       <visual>
         <origin xyz="0 0 0" rpy="0 0 0" />
         <geometry>
-          <mesh filename="${mesh_filename}" />
+          <mesh filename="${stl_mesh}" />
+        </geometry>
+      </visual>
+    </xacro:if>
+    <xacro:unless value="${use_gazebo_visual_meshes}">
+      <visual>
+        <origin xyz="0 0 0" rpy="0 0 0" />
+        <geometry>
+          <mesh filename="${dae_mesh}" />
         </geometry>
       </visual>
@@ -29,12 +23,7 @@
   </xacro:macro>
   <link name="ur10">
-    <xacro:ur_visual_or_gazebo_cylinder
-      mesh_filename="package://my_robot/meshes/base.dae"
-      radius="0.075"
-      length="0.038"
-      origin_xyz="0 0 0.019"
-      origin_rpy="0 0 0"
-      material_name="ur10_base_mat"
-      material_rgba="0.27 0.27 0.29 1.0" />
+    <xacro:ur_visual_mesh
+      dae_mesh="package://my_robot/meshes/base.dae"
+      stl_mesh="file://$(find my_robot)/meshes/base_gazebo_visual.stl" />
     <collision>
       <origin xyz="0 0 0.019" rpy="0 0 0" />
@@ -50,12 +39,7 @@
   </link>
   <link name="ur10_shoulder">
-    <xacro:ur_visual_or_gazebo_cylinder
-      mesh_filename="package://my_robot/meshes/shoulder.dae"
-      radius="0.075"
-      length="0.177"
-      origin_xyz="0 0 0"
-      origin_rpy="0 0 0"
-      material_name="ur10_shoulder_mat"
-      material_rgba="0.60 0.61 0.64 1.0" />
+    <xacro:ur_visual_mesh
+      dae_mesh="package://my_robot/meshes/shoulder.dae"
+      stl_mesh="file://$(find my_robot)/meshes/shoulder_gazebo_visual.stl" />
     <collision>
       <origin xyz="0 0 0" rpy="0 0 0" />
@@ -71,35 +55,7 @@
   </link>
   <link name="ur10_upper_arm">
-    <xacro:if value="${use_gazebo_compatible_visuals}">
-      <visual>
-        <origin xyz="0 -0.045 0" rpy="1.5707 0 0" />
-        <geometry>
-          <cylinder radius="0.075" length="0.177" />
-        </geometry>
-        <xacro:ur_gray_material name="ur10_upper_arm_head_mat" rgba="0.62 0.63 0.66 1.0" />
-      </visual>
-      <visual>
-        <origin xyz="0 -0.0436 0.32" rpy="0 0 1.5707" />
-        <geometry>
-          <cylinder radius="0.058" length="0.461" />
-        </geometry>
-        <xacro:ur_gray_material name="ur10_upper_arm_body_mat" rgba="0.76 0.76 0.79 1.0" />
-      </visual>
-      <visual>
-        <origin xyz="0 -0.04 0.613" rpy="1.5707 0 0" />
-        <geometry>
-          <cylinder radius="0.058" length="0.129" />
-        </geometry>
-        <xacro:ur_gray_material name="ur10_upper_arm_cap_mat" rgba="0.62 0.63 0.66 1.0" />
-      </visual>
-    </xacro:if>
-    <xacro:unless value="${use_gazebo_compatible_visuals}">
-      <visual>
-        <origin xyz="0 0 0" rpy="0 0 0" />
-        <geometry>
-          <mesh filename="package://my_robot/meshes/upperarm.dae" />
-        </geometry>
-      </visual>
-    </xacro:unless>
+    <xacro:ur_visual_mesh
+      dae_mesh="package://my_robot/meshes/upperarm.dae"
+      stl_mesh="file://$(find my_robot)/meshes/upperarm_gazebo_visual.stl" />
     <collision>
       <origin xyz="0 -0.045 0" rpy="1.5707 0 0" />
@@ -127,35 +83,7 @@
   </link>
   <link name="ur10_forearm">
-    <xacro:if value="${use_gazebo_compatible_visuals}">
-      <visual>
-        <origin xyz="0 0 0.001" rpy="1.5707 0 0" />
-        <geometry>
-          <cylinder radius="0.058" length="0.136" />
-        </geometry>
-        <xacro:ur_gray_material name="ur10_forearm_base_mat" rgba="0.62 0.63 0.66 1.0" />
-      </visual>
-      <visual>
-        <origin xyz="0 0 0.305" rpy="0 0 1.5707" />
-        <geometry>
-          <cylinder radius="0.045" length="0.447" />
-        </geometry>
-        <xacro:ur_gray_material name="ur10_forearm_body_mat" rgba="0.76 0.76 0.79 1.0" />
-      </visual>
-      <visual>
-        <origin xyz="0 0.001 0.5735" rpy="1.5707 0 0" />
-        <geometry>
-          <cylinder radius="0.045" length="0.119" />
-        </geometry>
-        <xacro:ur_gray_material name="ur10_forearm_cap_mat" rgba="0.62 0.63 0.66 1.0" />
-      </visual>
-    </xacro:if>
-    <xacro:unless value="${use_gazebo_compatible_visuals}">
-      <visual>
-        <origin xyz="0 0 0" rpy="0 0 0" />
-        <geometry>
-          <mesh filename="package://my_robot/meshes/forearm.dae" />
-        </geometry>
-      </visual>
-    </xacro:unless>
+    <xacro:ur_visual_mesh
+      dae_mesh="package://my_robot/meshes/forearm.dae"
+      stl_mesh="file://$(find my_robot)/meshes/forearm_gazebo_visual.stl" />
     <collision>
       <origin xyz="0 0 0.001" rpy="1.5707 0 0" />
@@ -183,12 +111,7 @@
   </link>
   <link name="ur10_wrist_1">
-    <xacro:ur_visual_or_gazebo_cylinder
-      mesh_filename="package://my_robot/meshes/wrist1.dae"
-      radius="0.0455"
-      length="0.119"
-      origin_xyz="0 0.115 0.0025"
-      origin_rpy="0 0 0"
-      material_name="ur10_wrist_1_mat"
-      material_rgba="0.58 0.59 0.62 1.0" />
+    <xacro:ur_visual_mesh
+      dae_mesh="package://my_robot/meshes/wrist1.dae"
+      stl_mesh="file://$(find my_robot)/meshes/wrist1_gazebo_visual.stl" />
     <collision>
       <origin xyz="0 0.115 0.0025" rpy="0 0 0" />
@@ -204,12 +127,7 @@
   </link>
   <link name="ur10_wrist_2">
-    <xacro:ur_visual_or_gazebo_cylinder
-      mesh_filename="package://my_robot/meshes/wrist2.dae"
-      radius="0.0455"
-      length="0.119"
-      origin_xyz="0 0.002 0.11659"
-      origin_rpy="1.5707 0 0"
-      material_name="ur10_wrist_2_mat"
-      material_rgba="0.58 0.59 0.62 1.0" />
+    <xacro:ur_visual_mesh
+      dae_mesh="package://my_robot/meshes/wrist2.dae"
+      stl_mesh="file://$(find my_robot)/meshes/wrist2_gazebo_visual.stl" />
     <collision>
       <origin xyz="0 0.002 0.11659" rpy="1.5707 0 0" />
@@ -225,12 +143,7 @@
   </link>
   <link name="ur10_wrist_3">
-    <xacro:ur_visual_or_gazebo_cylinder
-      mesh_filename="package://my_robot/meshes/wrist3.dae"
-      radius="0.045"
-      length="0.031"
-      origin_xyz="0 0.0765 0"
-      origin_rpy="1.5707 0 0"
-      material_name="ur10_wrist_3_mat"
-      material_rgba="0.58 0.59 0.62 1.0" />
+    <xacro:ur_visual_mesh
+      dae_mesh="package://my_robot/meshes/wrist3.dae"
+      stl_mesh="file://$(find my_robot)/meshes/wrist3_gazebo_visual.stl" />
     <collision>
       <origin xyz="0 0.0765 0" rpy="1.5707 0 0" />
@@ -245,11 +158,11 @@
     </inertial>
   </link>
-  <link name="铲子">
+  <link name="shovel_link">
     <visual>
       <origin xyz="0 0 0" rpy="0 0 0" />
       <geometry>
-        <mesh filename="package://my_robot/meshes/base_link.STL" />
-      </geometry>
-      <material name="铲子_mat">
+        <mesh filename="file://$(find my_robot)/meshes/base_link.STL" />
+      </geometry>
+      <material name="shovel_material">
         <color rgba="0.64706275 0.61961176 0.58823922 1.00000000"/>
       </material>
@@ -258,5 +171,5 @@
       <origin xyz="0 0 0" rpy="0 0 0" />
       <geometry>
-        <mesh filename="package://my_robot/meshes/base_link.STL" />
+        <mesh filename="file://$(find my_robot)/meshes/base_link.STL" />
       </geometry>
     </collision>
@@ -311,5 +224,5 @@
   <joint name="ur10-robot" type="fixed">
     <parent link="ur10_wrist_3" />
-    <child link="铲子" />
+    <child link="shovel_link" />
     <origin xyz="0 0.105 0" rpy="1.5707963 0 -1.5707963" />
   </joint>
@@ -524,5 +437,5 @@
       </xacro:if>
   </xacro:if>
-  <xacro:if value="${ros_profile == 'ros2' and ros_hardware_interface == 'effort'}">
+  <xacro:if value="${include_ros2_control == 'true' and ros_profile == 'ros2' and ros_hardware_interface == 'effort'}">
       <ros2_control name="my_robot" type="system">
         <hardware>
@@ -575,5 +488,5 @@
       </xacro:if>
   </xacro:if>
-  <xacro:if value="${ros_profile == 'ros2' and ros_hardware_interface == 'position'}">
+  <xacro:if value="${include_ros2_control == 'true' and ros_profile == 'ros2' and ros_hardware_interface == 'position'}">
       <ros2_control name="my_robot" type="system">
         <hardware>
@@ -620,5 +533,5 @@
       </xacro:if>
   </xacro:if>
-  <xacro:if value="${ros_profile == 'ros2' and ros_hardware_interface == 'velocity'}">
+  <xacro:if value="${include_ros2_control == 'true' and ros_profile == 'ros2' and ros_hardware_interface == 'velocity'}">
       <ros2_control name="my_robot" type="system">
         <hardware>

Commit message: Removes deprecated FT300 packages, improves MoveIt integration and launch system, adds executor parameter reconfiguration
- Deletes obsolete ft300_gui_ros2 and my_robotiq_force_torque_sensor packages, along with old driver files and zip archives.
- Adds default planner config (RRTConnect) for OMPL planning group and sets it in RViz config.
- Adds disable_collisions entries for gantry structure links against the arm and tool to avoid false collision checks in MoveIt.
- Fixes UR10 mount rotation in URDF (adds 90° rotation about Z axis).
- Updates full_system.launch.py: introduces `start_moveit` argument (default true), uses dedicated `gazebo_gantry.launch.py`, and launches MoveIt via a delayed `moveit_only.launch.py` to allow for staged startup.
- Removes `planner_mode` parameter from GUI node in the launch file.
- Adds runtime parameter reconfiguration to executor_node for `execution_mode`, `max_joint_step_rad`, and `dt` via `on_set_parameters` callback.
- Updates planner_node to deprecate non-`dp_rrt` modes, always falling back to dp_rrt; OMPL should be used via MoveIt/RViz.
- Updates bucket_scene_node to check `rclpy.ok()` before shutdown.
- Modifies package.xml of ur10_unified_gui to add `rcl_interfaces` and `moveit_msgs` dependencies.
- Updates README.md and full_system_upgrade_summary.md to reflect these changes and clarify two-stage launch workflow.

File: src/my_robot_moveit_config/srdf/my_robot.srdf.xacro (robot description, xacro)
@@ -46,3 +46,48 @@
   <disable_collisions link1="ur10_wrist_3" link2="shovel_tip" reason="Adjacent" />
   <disable_collisions link1="shovel_link" link2="shovel_tip" reason="Never" />
+  <!-- Ignore gantry-vs-arm/tool collision checks for planning -->
+  <disable_collisions link1="gantry_structure_link" link2="ur10" reason="Never" />
+  <disable_collisions link1="gantry_structure_link" link2="ur10_shoulder" reason="Never" />
+  <disable_collisions link1="gantry_structure_link" link2="ur10_upper_arm" reason="Never" />
+  <disable_collisions link1="gantry_structure_link" link2="ur10_forearm" reason="Never" />
+  <disable_collisions link1="gantry_structure_link" link2="ur10_wrist_1" reason="Never" />
+  <disable_collisions link1="gantry_structure_link" link2="ur10_wrist_2" reason="Never" />
+  <disable_collisions link1="gantry_structure_link" link2="ur10_wrist_3" reason="Never" />
+  <disable_collisions link1="gantry_structure_link" link2="shovel_link" reason="Never" />
+  <disable_collisions link1="gantry_structure_link" link2="shovel_tip" reason="Never" />
+  <disable_collisions link1="gantry_x_carriage_link" link2="ur10" reason="Never" />
+  <disable_collisions link1="gantry_x_carriage_link" link2="ur10_shoulder" reason="Never" />
+  <disable_collisions link1="gantry_x_carriage_link" link2="ur10_upper_arm" reason="Never" />
+  <disable_collisions link1="gantry_x_carriage_link" link2="ur10_forearm" reason="Never" />
+  <disable_collisions link1="gantry_x_carriage_link" link2="ur10_wrist_1" reason="Never" />
+  <disable_collisions link1="gantry_x_carriage_link" link2="ur10_wrist_2" reason="Never" />
+  <disable_collisions link1="gantry_x_carriage_link" link2="ur10_wrist_3" reason="Never" />
+  <disable_collisions link1="gantry_x_carriage_link" link2="shovel_link" reason="Never" />
+  <disable_collisions link1="gantry_x_carriage_link" link2="shovel_tip" reason="Never" />
+  <disable_collisions link1="gantry_y_carriage_link" link2="ur10" reason="Never" />
+  <disable_collisions link1="gantry_y_carriage_link" link2="ur10_shoulder" reason="Never" />
+  <disable_collisions link1="gantry_y_carriage_link" link2="ur10_upper_arm" reason="Never" />
+  <disable_collisions link1="gantry_y_carriage_link" link2="ur10_forearm" reason="Never" />
+  <disable_collisions link1="gantry_y_carriage_link" link2="ur10_wrist_1" reason="Never" />
+  <disable_collisions link1="gantry_y_carriage_link" link2="ur10_wrist_2" reason="Never" />
+  <disable_collisions link1="gantry_y_carriage_link" link2="ur10_wrist_3" reason="Never" />
+  <disable_collisions link1="gantry_y_carriage_link" link2="shovel_link" reason="Never" />
+  <disable_collisions link1="gantry_y_carriage_link" link2="shovel_tip" reason="Never" />
+  <disable_collisions link1="gantry_z_carriage_link" link2="ur10" reason="Never" />
+  <disable_collisions link1="gantry_z_carriage_link" link2="ur10_shoulder" reason="Never" />
+  <disable_collisions link1="gantry_z_carriage_link" link2="ur10_upper_arm" reason="Never" />
+  <disable_collisions link1="gantry_z_carriage_link" link2="ur10_forearm" reason="Never" />
+  <disable_collisions link1="gantry_z_carriage_link" link2="ur10_wrist_1" reason="Never" />
+  <disable_collisions link1="gantry_z_carriage_link" link2="ur10_wrist_2" reason="Never" />
+  <disable_collisions link1="gantry_z_carriage_link" link2="ur10_wrist_3" reason="Never" />
+  <disable_collisions link1="gantry_z_carriage_link" link2="shovel_link" reason="Never" />
+  <disable_collisions link1="gantry_z_carriage_link" link2="shovel_tip" reason="Never" />
+  <disable_collisions link1="ur_mount_link" link2="ur10_shoulder" reason="Never" />
+  <disable_collisions link1="ur_mount_link" link2="ur10_upper_arm" reason="Never" />
+  <disable_collisions link1="ur_mount_link" link2="ur10_forearm" reason="Never" />
+  <disable_collisions link1="ur_mount_link" link2="ur10_wrist_1" reason="Never" />
+  <disable_collisions link1="ur_mount_link" link2="ur10_wrist_2" reason="Never" />
+  <disable_collisions link1="ur_mount_link" link2="ur10_wrist_3" reason="Never" />
+  <disable_collisions link1="ur_mount_link" link2="shovel_link" reason="Never" />
+  <disable_collisions link1="ur_mount_link" link2="shovel_tip" reason="Never" />
 </robot>

File: src/my_robot_xacro/my_robot/urdf/my_robot_gantry.urdf.xacro (robot description, xacro)
@@ -195,5 +195,5 @@
     <parent link="ur_mount_link" />
     <child link="ur10" />
-    <origin xyz="0 0 -0.20" rpy="3.141592653589793 0 0" />
+    <origin xyz="0 0 -0.20" rpy="3.141592653589793 0 1.5707963267948966" />
   </joint>
   <xacro:my_robot_model
