Commit message: Updates URDF mesh paths and refines robot assembly config
- Parameterizes mesh file paths in assembly URDF using xacro argument for better flexibility
- Fixes joint naming consistency and corrects rotation values for sensor-shovel attachment
- Adjusts MoveIt trajectory execution start tolerance to improve motion planning reliability
- Disables simulation time for real hardware operation
- Removes temporary report file

File: src/ur_base_xarco_model/assembly_xacro/assembly/assembly.urdf.xacro (robot description, xacro)
@@ -1,11 +1,12 @@
 <?xml version="1.0"?>
 <robot name="assembly" xmlns:xacro="http://www.ros.org/wiki/xacro">
+  <xacro:arg name="mesh_root" default="meshes" />
   <link name="sensor_shovel">
     <visual>
       <origin xyz="0 0 0" rpy="0 0 0" />
       <geometry>
-        <mesh filename="meshes/base_link.STL" />
-      </geometry>
-      <material>
+        <mesh filename="$(arg mesh_root)/base_link.STL" />
+      </geometry>
+      <material name="mat_sensor_shovel">
         <color rgba="0.79216078 0.81961176 0.92941569 1.00000000"/>
       </material>
@@ -14,5 +15,5 @@
       <origin xyz="0 0 0" rpy="0 0 0" />
       <geometry>
-        <mesh filename="meshes/base_link.STL" />
+        <mesh filename="$(arg mesh_root)/base_link.STL" />
       </geometry>
     </collision>
@@ -23,11 +24,11 @@
     </inertial>
   </link>
-  <link name="sensor_shovel_shovel_tcp">
-    <visual>
-      <origin xyz="0 0 0" rpy="0 0 0" />
-      <geometry>
-        <mesh filename="meshes/shovel_tcp.STL" />
-      </geometry>
-      <material>
+  <link name="sensor_shovel_tcp">
+    <visual>
+      <origin xyz="0 0 0" rpy="0 0 0" />
+      <geometry>
+        <mesh filename="$(arg mesh_root)/shovel_tcp.STL" />
+      </geometry>
+      <material name="mat_shovel_tcp">
         <color rgba="1.00000000 1.00000000 1.00000000 1.00000000"/>
       </material>
@@ -36,5 +37,5 @@
       <origin xyz="0 0 0" rpy="0 0 0" />
       <geometry>
-        <mesh filename="meshes/shovel_tcp.STL" />
+        <mesh filename="$(arg mesh_root)/shovel_tcp.STL" />
       </geometry>
     </collision>
@@ -49,5 +50,5 @@
       <origin xyz="0 0 0" rpy="0 0 0" />
       <geometry>
-        <mesh filename="meshes/base.dae" />
+        <mesh filename="$(arg mesh_root)/base.dae" />
       </geometry>
       <material name="SWMaterial-2_001">
@@ -71,5 +72,5 @@
       <origin xyz="0 0 0" rpy="0 0 0" />
       <geometry>
-        <mesh filename="meshes/shoulder.dae" />
+        <mesh filename="$(arg mesh_root)/shoulder.dae" />
       </geometry>
       <material name="SWMaterial-0">
@@ -99,5 +100,5 @@
       <origin xyz="0 0 0" rpy="0 0 0" />
       <geometry>
-        <mesh filename="meshes/upperarm.dae" />
+        <mesh filename="$(arg mesh_root)/upperarm.dae" />
       </geometry>
       <material name="SWMaterial-0">
@@ -142,5 +143,5 @@
       <origin xyz="0 0 0" rpy="0 0 0" />
       <geometry>
-        <mesh filename="meshes/forearm.dae" />
+        <mesh filename="$(arg mesh_root)/forearm.dae" />
       </geometry>
       <material name="SWMaterial-0">
@@ -188,5 +189,5 @@
       <origin xyz="0 0 0" rpy="0 0 0" />
       <geometry>
-        <mesh filename="meshes/wrist1.dae" />
+        <mesh filename="$(arg mesh_root)/wrist1.dae" />
       </geometry>
       <material name="SWMaterial-0_001">
@@ -216,5 +217,5 @@
       <origin xyz="0 0 0" rpy="0 0 0" />
       <geometry>
-        <mesh filename="meshes/wrist2.dae" />
+        <mesh filename="$(arg mesh_root)/wrist2.dae" />
       </geometry>
       <material name="SWMaterial-0_002">
@@ -244,5 +245,5 @@
       <origin xyz="0 0 0" rpy="0 0 0" />
       <geometry>
-        <mesh filename="meshes/wrist3.dae" />
+        <mesh filename="$(arg mesh_root)/wrist3.dae" />
       </geometry>
       <material name="SWMaterial-2_003">
@@ -266,7 +267,7 @@
       <origin xyz="0 0 0" rpy="0 0 0" />
       <geometry>
-        <mesh filename="meshes/base_link_world_jizuo.STL" />
-      </geometry>
-      <material>
+        <mesh filename="$(arg mesh_root)/base_link_world_jizuo.STL" />
+      </geometry>
+      <material name="mat_base_jizuo">
         <color rgba="1.00000000 1.00000000 1.00000000 1.00000000"/>
       </material>
@@ -275,5 +276,5 @@
       <origin xyz="0 0 0" rpy="0 0 0" />
       <geometry>
-        <mesh filename="meshes/base_link_world_jizuo.STL" />
+        <mesh filename="$(arg mesh_root)/base_link_world_jizuo.STL" />
       </geometry>
     </collision>
@@ -288,7 +289,7 @@
       <origin xyz="0 0 0" rpy="0 0 0" />
       <geometry>
-        <mesh filename="meshes/base_ur10_with_dizuo.STL" />
-      </geometry>
-      <material>
+        <mesh filename="$(arg mesh_root)/base_ur10_with_dizuo.STL" />
+      </geometry>
+      <material name="mat_base_ur10_with_dizuo">
         <color rgba="1.00000000 1.00000000 1.00000000 1.00000000"/>
       </material>
@@ -297,5 +298,5 @@
       <origin xyz="0 0 0" rpy="0 0 0" />
       <geometry>
-        <mesh filename="meshes/base_ur10_with_dizuo.STL" />
+        <mesh filename="$(arg mesh_root)/base_ur10_with_dizuo.STL" />
       </geometry>
     </collision>
@@ -306,7 +307,7 @@
     </inertial>
   </link>
-  <joint name="sensor_shovel_tcp" type="fixed">
+  <joint name="sensor_shovel_tcp_fixed" type="fixed">
     <parent link="sensor_shovel" />
-    <child link="sensor_shovel_shovel_tcp" />
+    <child link="sensor_shovel_tcp" />
     <origin xyz="-0.47377 0.077109 0.0733" rpy="-1.5708 1.5708 -0.61087" />
   </joint>
@@ -361,7 +362,6 @@
     <parent link="ur10_wrist_3" />
     <child link="sensor_shovel" />
-    <origin xyz="0 0.09 0" rpy="-1.5707963 -1.5707963 0" quat_xyzw="-0.5 0.5 0.5 0.5" />
-  </joint>
-+
+    <origin xyz="0 0.09 0" rpy="-1.5707963 0 0" quat_xyzw="-0.5 0.5 0.5 0.5" />
+  </joint>
   <joint name="base_jizuo-ur10" type="fixed">
     <parent link="base_jizuo_base_ur10_with_dizuo" />
