Commit message: Updates UR10 real control with improved SRDF, URDF, and launch config
Fixes wrist link naming inconsistencies in URDF and SRDF to match standard UR10 conventions, replacing joint names with proper link names for wrist_1, wrist_2, and wrist_3. Adds collision pairs for the sensor shovel end effector.

Enables scaled joint trajectory controller as the default and configures reverse communication ports for real robot control. Adds a new real_control_gui.py script and its launcher to the install targets.

Improves robot readiness check script with ANSI stripping for cleaner controller status parsing and adds speed scaling topic verification to ensure the robot is properly initialized before execution.

Adjusts MoveIt RViz interactive marker size and relaxes trajectory execution start tolerance for more robust real-world operation. Adds launch_driver argument to allow conditional driver startup and makes RViz output visible on screen.

File: src/ur10_assembly_real_control/config/assembly_real.urdf.xacro (robot description, xacro)
@@ -185,5 +185,5 @@
     </inertial>
   </link>
-  <link name="wrist_1_joint">
+  <link name="wrist_1_link">
     <visual>
       <origin xyz="0 0 0" rpy="0 0 0" />
@@ -213,5 +213,5 @@
     </inertial>
   </link>
-  <link name="wrist_2_joint">
+  <link name="wrist_2_link">
     <visual>
       <origin xyz="0 0 0" rpy="0 0 0" />
@@ -241,5 +241,5 @@
     </inertial>
   </link>
-  <link name="wrist_3_joint">
+  <link name="wrist_3_link">
     <visual>
       <origin xyz="0 0 0" rpy="0 0 0" />
@@ -335,5 +335,5 @@
   <joint name="wrist_1_joint" type="revolute">
     <parent link="ur10_forearm" />
-    <child link="wrist_1_joint" />
+    <child link="wrist_1_link" />
     <origin xyz="-0.0000036 0 0.5723" rpy="0 1.5707895 0.0000027" />
     <axis xyz="0 1 0" />
@@ -341,6 +341,6 @@
   </joint>
   <joint name="wrist_2_joint" type="revolute">
-    <parent link="wrist_1_joint" />
-    <child link="wrist_2_joint" />
+    <parent link="wrist_1_link" />
+    <child link="wrist_2_link" />
     <origin xyz="0.0000003 0.1149 0.0000003" rpy="0 0 0" />
     <axis xyz="0 0 -1" />
@@ -348,6 +348,6 @@
   </joint>
   <joint name="wrist_3_joint" type="revolute">
-    <parent link="wrist_2_joint" />
-    <child link="wrist_3_joint" />
+    <parent link="wrist_2_link" />
+    <child link="wrist_3_link" />
     <origin xyz="0 -0.0000003 0.1157" rpy="0 0 0" />
     <axis xyz="0 1 0" />
@@ -360,5 +360,5 @@
   </joint>
   <joint name="ur10-sensor_shovel" type="fixed">
-    <parent link="wrist_3_joint" />
+    <parent link="wrist_3_link" />
     <child link="sensor_shovel" />
     <origin xyz="0 0.09 0" rpy="-1.5707963 0 0" quat_xyzw="-0.5 0.5 0.5 0.5" />

Commit message: Cleans up build artifacts and adds mud experiment recorder
Removes stale build/install/log directories and generated analysis outputs from version control to keep the repository clean. Adds comprehensive .gitignore rules for experiment data, data files, and ROS2 build artifacts.

Introduces a new mud experiment recorder package with core modules for UR10 control, FT300 force/torque sensor integration, RealSense camera recording, real-time weight calculation, and a PyQt5 GUI. Includes kinematics and dynamics estimation utilities for computing joint torques and force projections.

Adds MoveIt2 configuration for virtual UR10 assembly simulation with OMPL planning, ros2_control setup, and RViz2 visualization support. Updates the real UR10 launch configuration to properly load the custom assembly URDF and kinematics parameters.

Improves the WSLg compatibility for the dynamics measurement GUI by setting appropriate Wayland environment variables. Enhances the real UR10 readiness check script with RTDE overflow detection.

File: src/ur10_assembly_real_control/config/assembly_real.urdf.xacro (robot description, xacro)
@@ -1,5 +1,129 @@
 <?xml version="1.0"?>
 <robot name="assembly" xmlns:xacro="http://www.ros.org/wiki/xacro">
-  <xacro:arg name="mesh_root" default="meshes" />
+  <xacro:include filename="$(find ur_description)/urdf/ur_macro.xacro" />
+  <xacro:arg name="name" default="ur" />
+  <xacro:arg name="ur_type" default="ur10" />
+  <xacro:arg name="tf_prefix" default="" />
+  <xacro:arg name="mesh_root" default="file://$(find ur10_assembly_real_control)/config/meshes" />
+  <xacro:arg name="joint_limit_params" default="$(find ur10_assembly_real_control)/config/$(arg ur_type)/joint_limits.yaml" />
+  <xacro:arg name="kinematics_params" default="$(find ur10_assembly_real_control)/config/$(arg ur_type)/default_kinematics.yaml" />
+  <xacro:arg name="physical_params" default="$(find ur10_assembly_real_control)/config/$(arg ur_type)/physical_parameters.yaml" />
+  <xacro:arg name="visual_params" default="$(find ur10_assembly_real_control)/config/$(arg ur_type)/visual_parameters.yaml" />
+  <xacro:arg name="transmission_hw_interface" default="" />
+  <xacro:arg name="safety_limits" default="false" />
+  <xacro:arg name="safety_pos_margin" default="0.15" />
+  <xacro:arg name="safety_k_position" default="20" />
+  <xacro:arg name="headless_mode" default="false" />
+  <xacro:arg name="robot_ip" default="0.0.0.0" />
+  <xacro:arg name="script_filename" default="" />
+  <xacro:arg name="output_recipe_filename" default="" />
+  <xacro:arg name="input_recipe_filename" default="" />
+  <xacro:arg name="reverse_ip" default="0.0.0.0" />
+  <xacro:arg name="script_command_port" default="50004" />
+  <xacro:arg name="reverse_port" default="50001" />
+  <xacro:arg name="script_sender_port" default="50002" />
+  <xacro:arg name="trajectory_port" default="50003" />
+  <xacro:arg name="use_tool_communication" default="false" />
+  <xacro:arg name="tool_voltage" default="0" />
+  <xacro:arg name="tool_parity" default="0" />
+  <xacro:arg name="tool_baud_rate" default="115200" />
+  <xacro:arg name="tool_stop_bits" default="1" />
+  <xacro:arg name="tool_rx_idle_chars" default="1.5" />
+  <xacro:arg name="tool_tx_idle_chars" default="3.5" />
+  <xacro:arg name="tool_device_name" default="/tmp/ttyUR" />
+  <xacro:arg name="tool_tcp_port" default="54321" />
+  <xacro:arg name="use_fake_hardware" default="false" />
+  <xacro:arg name="fake_sensor_commands" default="false" />
+  <xacro:arg name="sim_gazebo" default="false" />
+  <xacro:arg name="sim_ignition" default="false" />
+  <xacro:arg name="initial_positions_file" default="$(find ur_description)/config/initial_positions.yaml" />
+  <xacro:property name="initial_positions_file" default="$(arg initial_positions_file)" />
+  <link name="base_jizuo">
+    <visual>
+      <origin xyz="0 0 0" rpy="0 0 0" />
+      <geometry>
+        <mesh filename="$(arg mesh_root)/base_link_world_jizuo.STL" />
+      </geometry>
+      <material name="mat_base_jizuo">
+        <color rgba="1.0 1.0 1.0 1.0" />
+      </material>
+    </visual>
+    <collision>
+      <origin xyz="0 0 0" rpy="0 0 0" />
+      <geometry>
+        <mesh filename="$(arg mesh_root)/base_link_world_jizuo.STL" />
+      </geometry>
+    </collision>
+    <inertial>
+      <origin xyz="-1.8696 -0.046752 0.24794" rpy="0 0 0" />
+      <mass value="1499.1" />
+      <inertia ixx="1126.8" ixy="-0.036857" ixz="0.0017432" iyy="2608.5" iyz="-18.236" izz="3614.6" />
+    </inertial>
+  </link>
+  <link name="base_jizuo_base_ur10_with_dizuo">
+    <visual>
+      <origin xyz="0 0 0" rpy="0 0 0" />
+      <geometry>
+        <mesh filename="$(arg mesh_root)/base_ur10_with_dizuo.STL" />
+      </geometry>
+      <material name="mat_base_ur10_with_dizuo">
+        <color rgba="1.0 1.0 1.0 1.0" />
+      </material>
+    </visual>
+    <collision>
+      <origin xyz="0 0 0" rpy="0 0 0" />
+      <geometry>
+        <mesh filename="$(arg mesh_root)/base_ur10_with_dizuo.STL" />
+      </geometry>
+    </collision>
+    <inertial>
+      <origin xyz="0 0 0.005" rpy="0 0 0" />
+      <mass value="0.225" />
+      <inertia ixx="0.0004237" ixy="0" ixz="0" iyy="0.0004237" iyz="0" izz="0.0008437" />
+    </inertial>
+  </link>
+  <joint name="base_jizuo_square_place" type="fixed">
+    <parent link="base_jizuo" />
+    <child link="base_jizuo_base_ur10_with_dizuo" />
+    <origin xyz="-0.78172 -0.025653 1.1638" rpy="3.1416 0 -1.5708" />
+  </joint>
+  <xacro:ur_robot
+    name="$(arg name)"
+    tf_prefix="$(arg tf_prefix)"
+    parent="base_jizuo_base_ur10_with_dizuo"
+    joint_limits_parameters_file="$(arg joint_limit_params)"
+    kinematics_parameters_file="$(arg kinematics_params)"
+    physical_parameters_file="$(arg physical_params)"
+    visual_parameters_file="$(arg visual_params)"
+    transmission_hw_interface="$(arg transmission_hw_interface)"
+    safety_limits="$(arg safety_limits)"
+    safety_pos_margin="$(arg safety_pos_margin)"
+    safety_k_position="$(arg safety_k_position)"
+    use_fake_hardware="$(arg use_fake_hardware)"
+    fake_sensor_commands="$(arg fake_sensor_commands)"
+    sim_gazebo="$(arg sim_gazebo)"
+    sim_ignition="$(arg sim_ignition)"
+    headless_mode="$(arg headless_mode)"
+    initial_positions="${xacro.load_yaml(initial_positions_file)}"
+    use_tool_communication="$(arg use_tool_communication)"
+    tool_voltage="$(arg tool_voltage)"
+    tool_parity="$(arg tool_parity)"
+    tool_baud_rate="$(arg tool_baud_rate)"
+    tool_stop_bits="$(arg tool_stop_bits)"
+    tool_rx_idle_chars="$(arg tool_rx_idle_chars)"
+    tool_tx_idle_chars="$(arg tool_tx_idle_chars)"
+    tool_device_name="$(arg tool_device_name)"
+    tool_tcp_port="$(arg tool_tcp_port)"
+    robot_ip="$(arg robot_ip)"
+    script_filename="$(arg script_filename)"
+    output_recipe_filename="$(arg output_recipe_filename)"
+    input_recipe_filename="$(arg input_recipe_filename)"
+    reverse_ip="$(arg reverse_ip)"
+    script_command_port="$(arg script_command_port)"
+    reverse_port="$(arg reverse_port)"
+    script_sender_port="$(arg script_sender_port)"
+    trajectory_port="$(arg trajectory_port)">
+    <origin xyz="0 0 0" rpy="0 0 0" />
+  </xacro:ur_robot>
   <link name="sensor_shovel">
     <visual>
@@ -9,5 +133,5 @@
       </geometry>
       <material name="mat_sensor_shovel">
-        <color rgba="0.79216078 0.81961176 0.92941569 1.00000000"/>
+        <color rgba="0.79216078 0.81961176 0.92941569 1.0" />
       </material>
     </visual>
@@ -31,5 +155,5 @@
       </geometry>
       <material name="mat_shovel_tcp">
-        <color rgba="1.00000000 1.00000000 1.00000000 1.00000000"/>
+        <color rgba="1.0 1.0 1.0 1.0" />
       </material>
     </visual>
@@ -40,271 +164,10 @@
       </geometry>
     </collision>
-    <inertial>
-      <origin xyz="0 -0.0002919 -0.00005" rpy="0 0 0" />
-      <mass value="0" />
-      <inertia ixx="0" ixy="0" ixz="0" iyy="0" iyz="0" izz="0" />
-    </inertial>
   </link>
-  <link name="ur10">
-    <visual>
-      <origin xyz="0 0 0" rpy="0 0 0" />
-      <geometry>
-        <mesh filename="$(arg mesh_root)/base.dae" />
-      </geometry>
-      <material name="SWMaterial-2_001">
-        <color rgba="0.37255294 0.37255294 0.37255294 1.00000000"/>
-      </material>
-    </visual>
-    <collision>
-      <origin xyz="0 0 0.019" rpy="0 0 0" />
-      <geometry>
-        <cylinder radius="0.075" length="0.038" />
-      </geometry>
-    </collision>
-    <inertial>
-      <origin xyz="0 0 0" rpy="0 0 0" />
-      <mass value="4" />
-      <inertia ixx="0.0061063" ixy="0" ixz="0" iyy="0.0061063" iyz="0" izz="0.01125" />
-    </inertial>
-  </link>
-  <link name="ur10_shoulder">
-    <visual>
-      <origin xyz="0 0 0" rpy="0 0 0" />
-      <geometry>
-        <mesh filename="$(arg mesh_root)/shoulder.dae" />
-      </geometry>
-      <material name="SWMaterial-0">
-        <color rgba="0.22353333 0.22353333 0.22353333 1.00000000"/>
-      </material>
-      <material name="SWMaterial-1">
-        <color rgba="0.39216078 0.54118039 0.63921961 1.00000000"/>
-      </material>
-      <material name="SWMaterial-2">
-        <color rgba="0.46274902 0.46274902 0.46274902 1.00000000"/>
-      </material>
-    </visual>
-    <collision>
-      <origin xyz="0 0 0" rpy="0 0 0" />
-      <geometry>
-        <cylinder radius="0.075" length="0.177" />
-      </geometry>
-    </collision>
-    <inertial>
-      <origin xyz="0 0 0" rpy="0 0 0" />
-      <mass value="7.778" />
-      <inertia ixx="0.0314743" ixy="0" ixz="0" iyy="0.0314743" iyz="0" izz="0.0218756" />
-    </inertial>
-  </link>
-  <link name="ur10_upper_arm">
-    <visual>
-      <origin xyz="0 0 0" rpy="0 0 0" />
-      <geometry>
-        <mesh filename="$(arg mesh_root)/upperarm.dae" />
-      </geometry>
-      <material name="SWMaterial-0">
-        <color rgba="0.22353333 0.22353333 0.22353333 1.00000000"/>
-      </material>
-      <material name="SWMaterial-1">
-        <color rgba="0.39216078 0.54118039 0.63921961 1.00000000"/>
-      </material>
-      <material name="SWMaterial-2">
-        <color rgba="0.46274902 0.46274902 0.46274902 1.00000000"/>
-      </material>
-      <material name="SWMaterial-3">
-        <color rgba="0.65490588 0.65490588 0.65490588 1.00000000"/>
-      </material>
-    </visual>
-    <collision>
-      <origin xyz="0 -0.045 0" rpy="1.5707 0 0" />
-      <geometry>
-        <cylinder radius="0.075" length="0.177" />
-      </geometry>
-    </collision>
-    <collision>
-      <origin xyz="0 -0.0436 0.32" rpy="0 0 1.5707" />
-      <geometry>
-        <cylinder radius="0.058" length="0.461" />
-      </geometry>
-    </collision>
-    <collision>
-      <origin xyz="0 -0.04 0.613" rpy="1.5707 0 0" />
-      <geometry>
-        <cylinder radius="0.058" length="0.129" />
-      </geometry>
-    </collision>
-    <inertial>
-      <origin xyz="0 0 0.306" rpy="0 0 0" />
-      <mass value="12.93" />
-      <inertia ixx="0.421754" ixy="0" ixz="0" iyy="0.421754" iyz="0" izz="0.0363656" />
-    </inertial>
-  </link>
-  <link name="ur10_forearm">
-    <visual>
-      <origin xyz="0 0 0" rpy="0 0 0" />
-      <geometry>
-        <mesh filename="$(arg mesh_root)/forearm.dae" />
-      </geometry>
-      <material name="SWMaterial-0">
-        <color rgba="0.22353333 0.22353333 0.22353333 1.00000000"/>
-      </material>
-      <material name="SWMaterial-1">
-        <color rgba="0.39216078 0.54118039 0.63921961 1.00000000"/>
-      </material>
-      <material name="SWMaterial-2">
-        <color rgba="0.46274902 0.46274902 0.46274902 1.00000000"/>
-      </material>
-      <material name="SWMaterial-3">
-        <color rgba="0.65490588 0.65490588 0.65490588 1.00000000"/>
-      </material>
-      <material name="SWMaterial-4">
-        <color rgba="0.07843529 0.07843529 0.07843529 1.00000000"/>
-      </material>
-    </visual>
-    <collision>
-      <origin xyz="0 0 0.001" rpy="1.5707 0 0" />
-      <geometry>
-        <cylinder radius="0.058" length="0.136" />
-      </geometry>
-    </collision>
-    <collision>
-      <origin xyz="0 0 0.305" rpy="0 0 1.5707" />
-      <geometry>
-        <cylinder radius="0.045" length="0.447" />
-      </geometry>
-    </collision>
-    <collision>
-      <origin xyz="0 0.001 0.5735" rpy="1.5707 0 0" />
-      <geometry>
-        <cylinder radius="0.045" length="0.119" />
-      </geometry>
-    </collision>
-    <inertial>
-      <origin xyz="0 0 0.28615" rpy="0 0 0" />
-      <mass value="3.87" />
-      <inertia ixx="0.11107" ixy="0" ixz="0" iyy="0.11107" iyz="0" izz="0.0108844" />
-    </inertial>
-  </link>
-  <link name="wrist_1_link">
-    <visual>
-      <origin xyz="0 0 0" rpy="0 0 0" />
-      <geometry>
-        <mesh filename="$(arg mesh_root)/wrist1.dae" />
-      </geometry>
-      <material name="SWMaterial-0_001">
-        <color rgba="0.22353333 0.22353333 0.22353333 1.00000000"/>
-      </material>
-      <material name="SWMaterial-1_001">
-        <color rgba="0.39216078 0.54118039 0.63921961 1.00000000"/>
-      </material>
-      <material name="SWMaterial-2_001">
-        <color rgba="0.46274902 0.46274902 0.46274902 1.00000000"/>
-      </material>
-    </visual>
-    <collision>
-      <origin xyz="0 0.115 0.0025" rpy="0 0 0" />
-      <geometry>
-        <cylinder radius="0.0455" length="0.119" />
-      </geometry>
-    </collision>
-    <inertial>
-      <origin xyz="0 0 0" rpy="0 0 0" />
-      <mass value="1.96" />
-      <inertia ixx="0.0051082" ixy="0" ixz="0" iyy="0.0051082" iyz="0" izz="0.0055125" />
-    </inertial>
-  </link>
-  <link name="wrist_2_link">
-    <visual>
-      <origin xyz="0 0 0" rpy="0 0 0" />
-      <geometry>
-        <mesh filename="$(arg mesh_root)/wrist2.dae" />
-      </geometry>
-      <material name="SWMaterial-0_002">
-        <color rgba="0.22353333 0.22353333 0.22353333 1.00000000"/>
-      </material>
-      <material name="SWMaterial-1_002">
-        <color rgba="0.39216078 0.54118039 0.63921961 1.00000000"/>
-      </material>
-      <material name="SWMaterial-2_002">
-        <color rgba="0.46274902 0.46274902 0.46274902 1.00000000"/>
-      </material>
-    </visual>
-    <collision>
-      <origin xyz="0 0.002 0.11659" rpy="1.5707 0 0" />
-      <geometry>
-        <cylinder radius="0.0455" length="0.119" />
-      </geometry>
-    </collision>
-    <inertial>
-      <origin xyz="0 0 0" rpy="0 0 0" />
-      <mass value="1.96" />
-      <inertia ixx="0.0051082" ixy="0" ixz="0" iyy="0.0051082" iyz="0" izz="0.0055125" />
-    </inertial>
-  </link>
-  <link name="wrist_3_link">
-    <visual>
-      <origin xyz="0 0 0" rpy="0 0 0" />
-      <geometry>
-        <mesh filename="$(arg mesh_root)/wrist3.dae" />
-      </geometry>
-      <material name="SWMaterial-2_003">
-        <color rgba="0.46274902 0.46274902 0.46274902 1.00000000"/>
-      </material>
-    </visual>
-    <collision>
-      <origin xyz="0 0.0765 0" rpy="1.5707 0 0" />
-      <geometry>
-        <cylinder radius="0.045" length="0.031" />
-      </geometry>
-    </collision>
-    <inertial>
-      <origin xyz="0 0 0" rpy="0 0 0" />
-      <mass value="0.202" />
-      <inertia ixx="0.0005265" ixy="0" ixz="0" iyy="0.0005265" iyz="0" izz="0.0005681" />
-    </inertial>
-  </link>
-  <link name="base_jizuo">
-    <visual>
-      <origin xyz="0 0 0" rpy="0 0 0" />
-      <geometry>
-        <mesh filename="$(arg mesh_root)/base_link_world_jizuo.STL" />
-      </geometry>
-      <material name="mat_base_jizuo">
-        <color rgba="1.00000000 1.00000000 1.00000000 1.00000000"/>
-      </material>
-    </visual>
-    <collision>
-      <origin xyz="0 0 0" rpy="0 0 0" />
-      <geometry>
-        <mesh filename="$(arg mesh_root)/base_link_world_jizuo.STL" />
-      </geometry>
-    </collision>
-    <inertial>
-      <origin xyz="-1.8696 -0.046752 0.24794" rpy="0 0 0" />
-      <mass value="1499.1" />
-      <inertia ixx="1126.8" ixy="-0.036857" ixz="0.0017432" iyy="2608.5" iyz="-18.236" izz="3614.6" />
-    </inertial>
-  </link>
-  <link name="base_jizuo_base_ur10_with_dizuo">
-    <visual>
-      <origin xyz="0 0 0" rpy="0 0 0" />
-      <geometry>
-        <mesh filename="$(arg mesh_root)/base_ur10_with_dizuo.STL" />
-      </geometry>
-      <material name="mat_base_ur10_with_dizuo">
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