Commit message: Switches to ur_base_xarco_model with renamed joints and mock hardware
Replaces the URDF model from the official ur_description package with the
custom ur_base_xarco_model assembly, preserving the original link/joint
naming and mesh structure. All joint names are updated from the standard
UR10 naming (e.g., shoulder_pan_joint) to the prefixed form
(ur10_shoulder_pan) throughout SRDF, joint limits, controllers, and
planning configuration.

Removes the now-unused config/ur10/ directory and initial_positions.yaml
to avoid stale references to the old joint names. The launch file is
simplified by dropping the ur_type argument and switching to the new
xacro parameters (ros_profile, ros_hardware_interface).

The ros2_control hardware plugin is replaced with mock_components/GenericSystem
to maintain a pure RViz2/MoveIt2 virtual control chain without Gazebo
dependencies. The readiness check script now includes retry logic with
short polling to avoid false negatives during startup.

File: src/ur10_assembly_virtual_moveit/urdf/assembly_virtual.urdf.xacro (robot description, xacro)
@@ -1,42 +1,266 @@
 <?xml version="1.0"?>
 <robot name="assembly" xmlns:xacro="http://www.ros.org/wiki/xacro">
-  <xacro:include filename="$(find ur_description)/urdf/ur_macro.xacro" />
-  <xacro:arg name="name" default="ur" />
-  <xacro:arg name="ur_type" default="ur10" />
-  <xacro:arg name="tf_prefix" default="" />
   <xacro:arg name="mesh_root" default="file://$(find ur10_assembly_virtual_moveit)/config/meshes" />
-  <xacro:arg name="joint_limit_params" default="$(find ur10_assembly_virtual_moveit)/config/$(arg ur_type)/joint_limits.yaml" />
-  <xacro:arg name="kinematics_params" default="$(find ur10_assembly_virtual_moveit)/config/$(arg ur_type)/default_kinematics.yaml" />
-  <xacro:arg name="physical_params" default="$(find ur10_assembly_virtual_moveit)/config/$(arg ur_type)/physical_parameters.yaml" />
-  <xacro:arg name="visual_params" default="$(find ur10_assembly_virtual_moveit)/config/$(arg ur_type)/visual_parameters.yaml" />
-  <xacro:arg name="transmission_hw_interface" default="" />
-  <xacro:arg name="safety_limits" default="false" />
-  <xacro:arg name="safety_pos_margin" default="0.15" />
-  <xacro:arg name="safety_k_position" default="20" />
-  <xacro:arg name="headless_mode" default="false" />
-  <xacro:arg name="robot_ip" default="0.0.0.0" />
-  <xacro:arg name="script_filename" default="" />
-  <xacro:arg name="output_recipe_filename" default="" />
-  <xacro:arg name="input_recipe_filename" default="" />
-  <xacro:arg name="reverse_ip" default="0.0.0.0" />
-  <xacro:arg name="script_command_port" default="50004" />
-  <xacro:arg name="reverse_port" default="50001" />
-  <xacro:arg name="script_sender_port" default="50002" />
-  <xacro:arg name="trajectory_port" default="50003" />
-  <xacro:arg name="use_tool_communication" default="false" />
-  <xacro:arg name="tool_voltage" default="0" />
-  <xacro:arg name="tool_parity" default="0" />
-  <xacro:arg name="tool_baud_rate" default="115200" />
-  <xacro:arg name="tool_stop_bits" default="1" />
-  <xacro:arg name="tool_rx_idle_chars" default="1.5" />
-  <xacro:arg name="tool_tx_idle_chars" default="3.5" />
-  <xacro:arg name="tool_device_name" default="/tmp/ttyUR" />
-  <xacro:arg name="tool_tcp_port" default="54321" />
-  <xacro:arg name="use_fake_hardware" default="true" />
-  <xacro:arg name="fake_sensor_commands" default="false" />
-  <xacro:arg name="sim_gazebo" default="false" />
-  <xacro:arg name="sim_ignition" default="false" />
-  <xacro:arg name="initial_positions_file" default="$(find ur_description)/config/initial_positions.yaml" />
-  <xacro:property name="initial_positions_file" default="$(arg initial_positions_file)" />
+  <link name="sensor_shovel">
+    <visual>
+      <origin xyz="0 0 0" rpy="0 0 0" />
+      <geometry>
+        <mesh filename="$(arg mesh_root)/base_link.STL" />
+      </geometry>
+      <material name="mat_sensor_shovel">
+        <color rgba="0.79216078 0.81961176 0.92941569 1.00000000"/>
+      </material>
+    </visual>
+    <collision>
+      <origin xyz="0 0 0" rpy="0 0 0" />
+      <geometry>
+        <mesh filename="$(arg mesh_root)/base_link.STL" />
+      </geometry>
+    </collision>
+    <inertial>
+      <origin xyz="-0.11585 0.0005511 0.051294" rpy="0 0 0" />
+      <mass value="2.3" />
+      <inertia ixx="0.0005331" ixy="0.0002664" ixz="0.0000158" iyy="0.0080026" iyz="0" izz="0.0082034" />
+    </inertial>
+  </link>
+  <link name="sensor_shovel_tcp">
+    <visual>
+      <origin xyz="0 0 0" rpy="0 0 0" />
+      <geometry>
+        <mesh filename="$(arg mesh_root)/shovel_tcp.STL" />
+      </geometry>
+      <material name="mat_shovel_tcp">
+        <color rgba="1.00000000 1.00000000 1.00000000 1.00000000"/>
+      </material>
+    </visual>
+    <collision>
+      <origin xyz="0 0 0" rpy="0 0 0" />
+      <geometry>
+        <mesh filename="$(arg mesh_root)/shovel_tcp.STL" />
+      </geometry>
+    </collision>
+    <inertial>
+      <origin xyz="0 -0.0002919 -0.00005" rpy="0 0 0" />
+      <mass value="0" />
+      <inertia ixx="0" ixy="0" ixz="0" iyy="0" iyz="0" izz="0" />
+    </inertial>
+  </link>
+  <link name="ur10">
+    <visual>
+      <origin xyz="0 0 0" rpy="0 0 0" />
+      <geometry>
+        <mesh filename="$(arg mesh_root)/base.dae" />
+      </geometry>
+      <material name="SWMaterial-2_001">
+        <color rgba="0.37255294 0.37255294 0.37255294 1.00000000"/>
+      </material>
+    </visual>
+    <collision>
+      <origin xyz="0 0 0.019" rpy="0 0 0" />
+      <geometry>
+        <cylinder radius="0.075" length="0.038" />
+      </geometry>
+    </collision>
+    <inertial>
+      <origin xyz="0 0 0" rpy="0 0 0" />
+      <mass value="4" />
+      <inertia ixx="0.0061063" ixy="0" ixz="0" iyy="0.0061063" iyz="0" izz="0.01125" />
+    </inertial>
+  </link>
+  <link name="ur10_shoulder">
+    <visual>
+      <origin xyz="0 0 0" rpy="0 0 0" />
+      <geometry>
+        <mesh filename="$(arg mesh_root)/shoulder.dae" />
+      </geometry>
+      <material name="SWMaterial-0">
+        <color rgba="0.22353333 0.22353333 0.22353333 1.00000000"/>
+      </material>
+      <material name="SWMaterial-1">
+        <color rgba="0.39216078 0.54118039 0.63921961 1.00000000"/>
+      </material>
+      <material name="SWMaterial-2">
+        <color rgba="0.46274902 0.46274902 0.46274902 1.00000000"/>
+      </material>
+    </visual>
+    <collision>
+      <origin xyz="0 0 0" rpy="0 0 0" />
+      <geometry>
+        <cylinder radius="0.075" length="0.177" />
+      </geometry>
+    </collision>
+    <inertial>
+      <origin xyz="0 0 0" rpy="0 0 0" />
+      <mass value="7.778" />
+      <inertia ixx="0.0314743" ixy="0" ixz="0" iyy="0.0314743" iyz="0" izz="0.0218756" />
+    </inertial>
+  </link>
+  <link name="ur10_upper_arm">
+    <visual>
+      <origin xyz="0 0 0" rpy="0 0 0" />
+      <geometry>
+        <mesh filename="$(arg mesh_root)/upperarm.dae" />
+      </geometry>
+      <material name="SWMaterial-0">
+        <color rgba="0.22353333 0.22353333 0.22353333 1.00000000"/>
+      </material>
+      <material name="SWMaterial-1">
+        <color rgba="0.39216078 0.54118039 0.63921961 1.00000000"/>
+      </material>
+      <material name="SWMaterial-2">
+        <color rgba="0.46274902 0.46274902 0.46274902 1.00000000"/>
+      </material>
+      <material name="SWMaterial-3">
+        <color rgba="0.65490588 0.65490588 0.65490588 1.00000000"/>
+      </material>
+    </visual>
+    <collision>
+      <origin xyz="0 -0.045 0" rpy="1.5707 0 0" />
+      <geometry>
+        <cylinder radius="0.075" length="0.177" />
+      </geometry>
+    </collision>
+    <collision>
+      <origin xyz="0 -0.0436 0.32" rpy="0 0 1.5707" />
+      <geometry>
+        <cylinder radius="0.058" length="0.461" />
+      </geometry>
+    </collision>
+    <collision>
+      <origin xyz="0 -0.04 0.613" rpy="1.5707 0 0" />
+      <geometry>
+        <cylinder radius="0.058" length="0.129" />
+      </geometry>
+    </collision>
+    <inertial>
+      <origin xyz="0 0 0.306" rpy="0 0 0" />
+      <mass value="12.93" />
+      <inertia ixx="0.421754" ixy="0" ixz="0" iyy="0.421754" iyz="0" izz="0.0363656" />
+    </inertial>
+  </link>
+  <link name="ur10_forearm">
+    <visual>
+      <origin xyz="0 0 0" rpy="0 0 0" />
+      <geometry>
+        <mesh filename="$(arg mesh_root)/forearm.dae" />
+      </geometry>
+      <material name="SWMaterial-0">
+        <color rgba="0.22353333 0.22353333 0.22353333 1.00000000"/>
+      </material>
+      <material name="SWMaterial-1">
+        <color rgba="0.39216078 0.54118039 0.63921961 1.00000000"/>
+      </material>
+      <material name="SWMaterial-2">
+        <color rgba="0.46274902 0.46274902 0.46274902 1.00000000"/>
+      </material>
+      <material name="SWMaterial-3">
+        <color rgba="0.65490588 0.65490588 0.65490588 1.00000000"/>
+      </material>
+      <material name="SWMaterial-4">
+        <color rgba="0.07843529 0.07843529 0.07843529 1.00000000"/>
+      </material>
+    </visual>
+    <collision>
+      <origin xyz="0 0 0.001" rpy="1.5707 0 0" />
+      <geometry>
+        <cylinder radius="0.058" length="0.136" />
+      </geometry>
+    </collision>
+    <collision>
+      <origin xyz="0 0 0.305" rpy="0 0 1.5707" />
+      <geometry>
+        <cylinder radius="0.045" length="0.447" />
+      </geometry>
+    </collision>
+    <collision>
+      <origin xyz="0 0.001 0.5735" rpy="1.5707 0 0" />
+      <geometry>
+        <cylinder radius="0.045" length="0.119" />
+      </geometry>
+    </collision>
+    <inertial>
+      <origin xyz="0 0 0.28615" rpy="0 0 0" />
+      <mass value="3.87" />
+      <inertia ixx="0.11107" ixy="0" ixz="0" iyy="0.11107" iyz="0" izz="0.0108844" />
+    </inertial>
+  </link>
+  <link name="ur10_wrist_1">
+    <visual>
+      <origin xyz="0 0 0" rpy="0 0 0" />
+      <geometry>
+        <mesh filename="$(arg mesh_root)/wrist1.dae" />
+      </geometry>
+      <material name="SWMaterial-0_001">
+        <color rgba="0.22353333 0.22353333 0.22353333 1.00000000"/>
+      </material>
+      <material name="SWMaterial-1_001">
+        <color rgba="0.39216078 0.54118039 0.63921961 1.00000000"/>
+      </material>
+      <material name="SWMaterial-2_001">
+        <color rgba="0.46274902 0.46274902 0.46274902 1.00000000"/>
+      </material>
+    </visual>
+    <collision>
+      <origin xyz="0 0.115 0.0025" rpy="0 0 0" />
+      <geometry>
+        <cylinder radius="0.0455" length="0.119" />
+      </geometry>
+    </collision>
+    <inertial>
+      <origin xyz="0 0 0" rpy="0 0 0" />
+      <mass value="1.96" />
+      <inertia ixx="0.0051082" ixy="0" ixz="0" iyy="0.0051082" iyz="0" izz="0.0055125" />
+    </inertial>
+  </link>
+  <link name="ur10_wrist_2">
+    <visual>
+      <origin xyz="0 0 0" rpy="0 0 0" />
+      <geometry>
+        <mesh filename="$(arg mesh_root)/wrist2.dae" />
+      </geometry>
+      <material name="SWMaterial-0_002">
+        <color rgba="0.22353333 0.22353333 0.22353333 1.00000000"/>
+      </material>
+      <material name="SWMaterial-1_002">
+        <color rgba="0.39216078 0.54118039 0.63921961 1.00000000"/>
+      </material>
+      <material name="SWMaterial-2_002">
+        <color rgba="0.46274902 0.46274902 0.46274902 1.00000000"/>
+      </material>
+    </visual>
+    <collision>
+      <origin xyz="0 0.002 0.11659" rpy="1.5707 0 0" />
+      <geometry>
+        <cylinder radius="0.0455" length="0.119" />
+      </geometry>
+    </collision>
+    <inertial>
+      <origin xyz="0 0 0" rpy="0 0 0" />
+      <mass value="1.96" />
+      <inertia ixx="0.0051082" ixy="0" ixz="0" iyy="0.0051082" iyz="0" izz="0.0055125" />
+    </inertial>
+  </link>
+  <link name="ur10_wrist_3">
+    <visual>
+      <origin xyz="0 0 0" rpy="0 0 0" />
+      <geometry>
+        <mesh filename="$(arg mesh_root)/wrist3.dae" />
+      </geometry>
+      <material name="SWMaterial-2_003">
+        <color rgba="0.46274902 0.46274902 0.46274902 1.00000000"/>
+      </material>
+    </visual>
+    <collision>
+      <origin xyz="0 0.0765 0" rpy="1.5707 0 0" />
+      <geometry>
+        <cylinder radius="0.045" length="0.031" />
+      </geometry>
+    </collision>
+    <inertial>
+      <origin xyz="0 0 0" rpy="0 0 0" />
+      <mass value="0.202" />
+      <inertia ixx="0.0005265" ixy="0" ixz="0" iyy="0.0005265" iyz="0" izz="0.0005681" />
+    </inertial>
+  </link>
   <link name="base_jizuo">
     <visual>
@@ -46,5 +270,5 @@
       </geometry>
       <material name="mat_base_jizuo">
-        <color rgba="1.0 1.0 1.0 1.0" />
+        <color rgba="1.00000000 1.00000000 1.00000000 1.00000000"/>
       </material>
     </visual>
@@ -68,5 +292,5 @@
       </geometry>
       <material name="mat_base_ur10_with_dizuo">
-        <color rgba="1.0 1.0 1.0 1.0" />
+        <color rgba="1.00000000 1.00000000 1.00000000 1.00000000"/>
       </material>
     </visual>
@@ -83,4 +307,51 @@
     </inertial>
   </link>
+  <joint name="sensor_shovel_tcp_fixed" type="fixed">
+    <parent link="sensor_shovel" />
+    <child link="sensor_shovel_tcp" />
+    <origin xyz="-0.47377 0.077109 0.0733" rpy="-1.5708 1.5708 -0.61087" />
+  </joint>
+  <joint name="ur10_shoulder_pan" type="revolute">
+    <parent link="ur10" />
+    <child link="ur10_shoulder" />
+    <origin xyz="0 0 0.1273" rpy="0 0 0" />
+    <axis xyz="0 0 1" />
+    <limit lower="-6.28319" upper="6.28319" effort="330" velocity="2.16" />
+  </joint>
+  <joint name="ur10_shoulder_lift" type="revolute">
+    <parent link="ur10_shoulder" />
+    <child link="ur10_upper_arm" />
+    <origin xyz="0 0.220941 0" rpy="0 1.57079 0" />
+    <axis xyz="0 1 0" />
+    <limit lower="-6.28319" upper="6.28319" effort="330" velocity="2.16" />
+  </joint>
+  <joint name="ur10_elbow" type="revolute">
+    <parent link="ur10_upper_arm" />
+    <child link="ur10_forearm" />
+    <origin xyz="-0.0000039 -0.1719 0.612" rpy="0 0 0" />
+    <axis xyz="0 1 0" />
+    <limit lower="-6.28319" upper="6.28319" effort="150" velocity="3.15" />
+  </joint>
+  <joint name="ur10_wrist_1" type="revolute">
+    <parent link="ur10_forearm" />
+    <child link="ur10_wrist_1" />
+    <origin xyz="-0.0000036 0 0.5723" rpy="0 1.5707895 0.0000027" />
+    <axis xyz="0 1 0" />
+    <limit lower="-6.28319" upper="6.28319" effort="54" velocity="3.2" />
+  </joint>
+  <joint name="ur10_wrist_2" type="revolute">
+    <parent link="ur10_wrist_1" />
+    <child link="ur10_wrist_2" />
+    <origin xyz="0.0000003 0.1149 0.0000003" rpy="0 0 0" />
+    <axis xyz="0 0 -1" />
+    <limit lower="-6.28319" upper="6.28319" effort="54" velocity="3.2" />
+  </joint>
+  <joint name="ur10_wrist_3" type="revolute">
+    <parent link="ur10_wrist_2" />
+    <child link="ur10_wrist_3" />
+    <origin xyz="0 -0.0000003 0.1157" rpy="0 0 0" />
+    <axis xyz="0 1 0" />
+    <limit lower="-6.28319" upper="6.28319" effort="54" velocity="3.2" />
+  </joint>
   <joint name="base_jizuo_square_place" type="fixed">
     <parent link="base_jizuo" />
@@ -88,90 +359,392 @@
     <origin xyz="-0.78172 -0.025653 1.1638" rpy="3.1416 0 -1.5708" />
   </joint>
-  <xacro:ur_robot
-    name="$(arg name)"
-    tf_prefix="$(arg tf_prefix)"
-    parent="base_jizuo_base_ur10_with_dizuo"
-    joint_limits_parameters_file="$(arg joint_limit_params)"
-    kinematics_parameters_file="$(arg kinematics_params)"
-    physical_parameters_file="$(arg physical_params)"
-    visual_parameters_file="$(arg visual_params)"
-    transmission_hw_interface="$(arg transmission_hw_interface)"
-    safety_limits="$(arg safety_limits)"
-    safety_pos_margin="$(arg safety_pos_margin)"
-    safety_k_position="$(arg safety_k_position)"
-    use_fake_hardware="$(arg use_fake_hardware)"
-    fake_sensor_commands="$(arg fake_sensor_commands)"
-    sim_gazebo="$(arg sim_gazebo)"
-    sim_ignition="$(arg sim_ignition)"
-    headless_mode="$(arg headless_mode)"
-    initial_positions="${xacro.load_yaml(initial_positions_file)}"
-    use_tool_communication="$(arg use_tool_communication)"
-    tool_voltage="$(arg tool_voltage)"
-    tool_parity="$(arg tool_parity)"
-    tool_baud_rate="$(arg tool_baud_rate)"
-    tool_stop_bits="$(arg tool_stop_bits)"
-    tool_rx_idle_chars="$(arg tool_rx_idle_chars)"
-    tool_tx_idle_chars="$(arg tool_tx_idle_chars)"
-    tool_device_name="$(arg tool_device_name)"
-    tool_tcp_port="$(arg tool_tcp_port)"
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